File: lead_acid_bms_hardware/lead_acid_bms_hardware.kicad_pcb (KiCad board)
At the start: 2 copper layers, 88 x 52.3 mm, 75 parts, among them J1 debugging_connector, J2 battery_p, J3 battery_n, J4 bms_p, J5 bms_n, Q1 IRFZ44N, Q10 CJ2305, Q11 CJ2305, Q2 IRFZ44N, Q3 MMBT3904, Q4 CJ2305, Q5 MMBT3904, Q6 S9015, Q7 MMBT3904, Q8 MMBT3904, Q9 S9015, SW1 rst, U1 AMS1117-3.3, U2 TL974IDR, U3 ATmega8-16A, U4 NRF24L01_Breakout

Commit message: Routing...
Parts:
- U2: moved to B.Cu
- moved R26 143.8 mm to (248.4, 61.7), turned to 0 degrees
- moved R35 136.7 mm to (92.0, 79.4), turned to 180 degrees
- moved U1 135.7 mm to (99.0, 88.5)
- moved R34 132.9 mm to (92.0, 71.6), turned to 180 degrees
- moved J4 123.4 mm to (162.5, 105.0)
- moved R1 116.6 mm to (108.4, 69.9), turned to -90 degrees
- moved R2 116.4 mm to (110.4, 69.9), turned to 90 degrees
- moved C1 109.6 mm to (91.5, 87.5), turned to -90 degrees
- moved R28 106.7 mm to (123.5, 51.3)
- moved C2 105.5 mm to (106.3, 67.3), turned to -90 degrees
- moved R7 103.2 mm to (126.4, 71.0), turned to -90 degrees
- moved Q11 102.5 mm to (245.9, 55.0)
- moved R36 102.3 mm to (109.2, 81.6)
- moved D2 101.7 mm to (92.0, 77.0)
- moved R29 101.3 mm to (123.7, 58.1)
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Routing:
- net +3V3: track 0.00 -> 39.4 mm
- net PROG_SCK: track 0.00 -> 35.2 mm, vias 0 -> 1
- net PROG_MISO: track 0.00 -> 30.8 mm, vias 0 -> 1
- net MCU_RST: track 0.00 -> 29.2 mm, vias 0 -> 1
- net PROG_MOSI: track 0.00 -> 27.3 mm, vias 0 -> 1
- net AVR_RX: track 0.00 -> 26.9 mm, vias 0 -> 1
- net AVR_TX: track 0.00 -> 26.7 mm, vias 0 -> 1
- net HIGH_SIDE_SENSE: track 11.7 -> 25.7 mm
- net VREF: track 0.00 -> 7.64 mm, vias 0 -> 1
- net LED1: track 0.00 -> 5.18 mm
- net LED2: track 0.00 -> 4.02 mm
- net Net-(D3-Pad1): track 0.00 -> 2.68 mm
- net Net-(D2-Pad1): track 0.00 -> 2.60 mm
- net Net-(D1-Pad1): track 0.00 -> 2.60 mm
- net SWITCHED_3V3: track 0.00 -> 2.41 mm
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- added copper zone on B.Cu, net BATTERY_N
- added copper zone on F.Cu, net BATTERY_N
- added copper zone on B.Cu, net BATTERY_P
- added copper zone on F.Cu, net BATTERY_P
- added copper zone on B.Cu, net BMS_N
- added copper zone on F.Cu, net BMS_N
Other:
- board size 88 x 52.3 mm -> 80 x 50 mm

Commit message: Almost done with PCB placement/routing. Need to find lower power amplifier (TL974IDR is not good enough)
Parts:
- removed the R1 at (108.4, 69.9)
- removed the R12 at (260.6, 53.9)
- removed the R5 at (121.4, 70.9)
- added R15: 100k, Resistor_SMD:R_0805_2012Metric, F.Cu at (258.4, 130.5)
- added R3: 100k, Resistor_SMD:R_0805_2012Metric, F.Cu at (253.9, 130.5)
- added R9: 100k, Resistor_SMD:R_0805_2012Metric, F.Cu at (253.9, 124.6)
- R13, R14, R2, R6, R7, R8: value 10k -> 100k
- U3: renamed from U2; moved to F.Cu
- moved R2 158.8 mm to (258.4, 127.5), turned to 0 degrees
- moved R6 151.9 mm to (262.8, 130.5), turned to 0 degrees
- moved R7 146.5 mm to (262.8, 124.6), turned to 0 degrees
- moved R8 146.1 mm to (262.8, 127.5), turned to 0 degrees
- moved Q4 129.4 mm to (102.2, 67.5)
- moved U3 121.2 mm to (213.0, 131.0), turned to 180 degrees
- moved R40 119.4 mm to (112.7, 89.5), turned to -90 degrees
- moved Q9 116.5 mm to (144.0, 96.3), turned to 180 degrees
- moved C2 112.5 mm to (202.1, 126.4)
- moved R30 111.5 mm to (211.9, 126.2), turned to 90 degrees
- moved R31 110.7 mm to (208.1, 135.8), turned to 90 degrees
- moved Q10 102.8 mm to (126.2, 97.3)
- moved Q8 99.0 mm to (147.9, 96.3), turned to 180 degrees
- moved R21 98.0 mm to (151.7, 97.0), turned to 180 degrees
- moved SW1 97.1 mm to (115.6, 98.5), turned to 180 degrees
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- renumbered C7 to C5, C8 to C6, C5 to C7, C6 to C8, R42 to R1, R9 to R10, R10 to R11, R11 to R12, R15 to R16, R16 to R17, R17 to R18, R18 to R19, R19 to R20, R20 to R21, R21 to R22, R22 to R23, R23 to R24, R24 to R25, R25 to R26, R26 to R27, R27 to R28, R28 to R29, R29 to R30, R30 to R31, R31 to R32, R32 to R33, R33 to R34, R34 to R35, R35 to R36, R36 to R37, R37 to R38, R38 to R39, R3 to R4, R39 to R40, R40 to R41, R41 to R42, R4 to R5, U1 to U2, U3 to U4, U4 to U5
Connections:
- R13 pad 1: Net-(R12-Pad2) -> BATTERY_P
- R13 pad 2: BAT_SENSE -> Net-(R13-Pad2)
- R14 pad 1: BAT_SENSE -> Net-(R13-Pad2)
- R14 pad 2: BATTERY_N -> BAT_SENSE
- R2 pad 1: VREF -> +3V3
- R2 pad 2: BATTERY_N -> VREF
- R6 pad 1: LOW_SIDE_SENSE_BIASED -> +3V3
- R6 pad 2: BATTERY_N -> LOW_SIDE_SENSE_BIASED
- R7 pad 1: SWITCHED_3V3 -> LOW_SIDE_SENSE_BIASED
- R7 pad 2: HIGH_SIDE_SENSE_BIASED -> BATTERY_N
- R8 pad 1: HIGH_SIDE_SENSE_BIASED -> +3V3
- R8 pad 2: HIGH_SIDE_SENSE -> HIGH_SIDE_SENSE_BIASED
Routing:
- net BATTERY_N: track 0.00 -> 61.8 mm
- net DFET_GATE_CTRL: track 0.00 -> 51.4 mm, vias 0 -> 2
- net SWITCHED_BATTERY_P: track 0.00 -> 30.8 mm, vias 0 -> 3
- net CHARGE_MOS_GATE: track 0.00 -> 21.4 mm, vias 0 -> 1
- net DISCHARGE_MOS_GATE: track 0.00 -> 20.6 mm, vias 0 -> 1
- net Net-(R28-Pad2): track 0.00 -> 9.15 mm
- net Net-(R27-Pad2): track 0.00 -> 8.96 mm
- net HIGH_RANGE_ANALOG_OUT: track 0.00 -> 8.31 mm
- net MCU_RST: track 29.2 -> 37.2 mm
- net Net-(Q3-Pad3): track 0.00 -> 8.01 mm
- net VREF: track 7.64 -> 0.00 mm, vias 1 -> 0
- net Net-(Q7-Pad3): track 0.00 -> 7.43 mm
- net Net-(R25-Pad2): track 0.00 -> 6.52 mm
- net Net-(R26-Pad2): track 0.00 -> 6.37 mm
- net Net-(R24-Pad2): track 0.00 -> 6.04 mm
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